File: project/file595D27E9.sch (KiCad schematic (older format))
At the start: 7 parts

Commit message: Add digital potentiometer (TPL0102-100) to schematic.
Parts:
- U?: footprint MODULE -> Housings_SSOP:TSSOP-16_4.4x5mm_Pitch0.65mm
Changed lines of the file:
@@
 $Descr A4 11693 8268
 encoding utf-8
-Sheet 6 6
+Sheet 6 7
 Title ""
 Date ""
@@
 F 0 "U?" H 5700 3650 50  0000 C CNN
 F 1 "AD5689R" H 5700 3850 50  0000 C CNN
-F 2 "MODULE" H 5700 3750 50  0001 C CNN
+F 2 "Housings_SSOP:TSSOP-16_4.4x5mm_Pitch0.65mm" H 5700 3750 50  0001 C CNN
 F 3 "DOCUMENTATION" H 5700 3750 50  0001 C CNN
 	1    5700 3750
